File: hardware/power.sch (KiCad schematic (older format))
At the start: 44 parts, among them Q3 FDV301N, Q4 FDV301N, Q5 DMP2120U, Q6 DMP2120U, U4 NCP700BSN30T1G, U5 MCP1501T-25E, U6 LM5164DDAR, U7 LM63615-Q1PWP

Commit message: Update BOM * Datasheets * Manufacturers * Part numbers
Parts:
- C20: Manufacturer (none) -> Taiyo Yuden; Model C3225X7R2A225K230AB -> (none); Part Number (none) -> HMK325B7225KM-T; Tolerance (none) -> 10%
- C21, C34: Manufacturer (none) -> Taiyo Yuden; Part Number (none) -> GMK316AB7106KL-TR; Tolerance (none) -> 10%
- C22, C25, C27, C36, C37: Manufacturer (none) -> KEMET; Part Number (none) -> C1206C105K3RACAUTO; Tolerance (none) -> 10%
- C23, C28: DNP (none) -> X; Manufacturer (none) -> KEMET; Part Number (none) -> C1206C105K3RACAUTO; Tolerance (none) -> 10%
- C24, C31: Manufacturer (none) -> TDK; Part Number (none) -> C1608X7R1H224K080AB; Tolerance (none) -> 10%
- C26, C35: Manufacturer (none) -> Taiyo Yuden; Part Number (none) -> GMK107B7104KAHT; Tolerance (none) -> 10%
- C29, C30: Manufacturer (none) -> KEMET; Model C0805C222K5RACTU -> (none); Part Number (none) -> C0805C222K5RACTU; Tolerance (none) -> 10%
- C32: Manufacturer (none) -> Wurth Electronik; Part Number (none) -> 885012006021; Tolerance (none) -> 5%; Voltage Rating (none) -> 16V
- C33: Manufacturer (none) -> Murata; Part Number (none) -> GRM32EC81C476KE15K; Tolerance (none) -> 10%
- JP2: DNP (none) -> X
- L2: Manufacturer (none) -> Coilcraft; Model MSS1210-104KEB -> (none); Part Number (none) -> MSS1210-104KEB
- L3: Manufacturer (none) -> TDK; Model SLF10165T-150M3R13PF -> (none); Part Number (none) -> SLF10165T-150M3R13PF
- Q3, Q4: Manufacturer (none) -> ON Semiconductor; Part Number (none) -> FDV301N
- Q5, Q6: Manufacturer (none) -> Diodes Incorporated; Part Number (none) -> DMP2120U
- R22: Manufacturer (none) -> Panasonic; Part Number (none) -> ERJ-3EKF2004V
- R23: Manufacturer (none) -> Stackpole Electronics Inc; Part Number (none) -> RMCF0603FT205K
- R24, R25: Manufacturer (none) -> Stackpole Electronics Inc; Part Number (none) -> RMCF0603FT150K
- R26: Manufacturer (none) -> Stackpole Electronics Inc; Part Number (none) -> RMCF0603FT39K2
- R27: DNP (none) -> X; Manufacturer (none) -> Stackpole Electronics Inc; Part Number (none) -> RMCF0603FT47R0; Tolerance 5% -> 1%
- R28: Manufacturer (none) -> Stackpole Electronics Inc; Part Number (none) -> RMCF0603FT270K
- R29: Manufacturer (none) -> Stackpole Electronics Inc; Part Number (none) -> RMCF0603FT536K
- R30: Manufacturer (none) -> Stackpole Electronics Inc; Part Number (none) -> RMCF0603FT59K0
- R31, R32: Manufacturer (none) -> Stackpole Electronics Inc; Part Number (none) -> RMCF0603FT47R0; Tolerance 5% -> 1%
- R33, R34: Manufacturer (none) -> Stackpole Electronics Inc; Part Number (none) -> RMCF0603JG10K0
- R35, R36: Manufacturer (none) -> Bourns; Part Number (none) -> CR0603-JW-473ELF
- U4: Manufacturer (none) -> ON Semiconductor; Part Number (none) -> NCP700BSN30T1G
- U5: DNP (none) -> X; Manufacturer (none) -> Microchip; Part Number (none) -> MCP1501T-25E/CHY
- U6: Manufacturer (none) -> Texas Instruments; Part Number (none) -> LM5164DDAR
- U7: Manufacturer (none) -> Texas Instruments; Part Number (none) -> LM63615-Q1PWP
