File: hardware/station.kicad_pcb (KiCad board)
At the start: 2 copper layers, 100 x 60 mm, 168 parts, among them J1 AudioJack3, J2 AudioJack3, J3 Conn_02x05_Odd_Even, J4 Conn_02x05_Counter_Clockwise, J5 Screw_Terminal_01x02, Q1 NTMFS5C682NL, Q2 NTMFS5C682NL, Q3 FDV301N, Q4 FDV301N, Q5 DMP2120U, Q6 DMP2120U, Q7 NTMFS5C682NL, Q8 NTMFS5C682NL, U1 NCS213, U10 LM5109BSD, U11 STM32G431CBT6, U2 MAX44246, U3 LM5109BSD, U4 NCP700BSN30T1G, U5 MCP1501T-25E, U6 LM5164DDAR, U7 LM63615-Q1PWP, U8 NCS213, U9 MAX44246

Commit message: Update BOM * Datasheets * Manufacturers * Part numbers
Parts:
- C1, C38, C4, C41, C45, C8: value DNF -> ?
- C17, C54: value 160n -> 150n
