File: hardware/station.sch (KiCad schematic (older format))
At the start: 5 parts, among them J1 AudioJack3, J2 AudioJack3, J3 Conn_02x05_Odd_Even

Commit message: Layout almost complete. Just needs a tidy.
Parts:
- added F1: Fuse, station:Fuse_2410, symbol Device:Fuse
- added F2: Fuse, Fuse:Fuse_1206_3216Metric, symbol Device:Fuse
- added J5: Screw_Terminal_01x02, TerminalBlock:TerminalBlock_bornier-2_P5.08mm, symbol Connector:Screw_Terminal_01x02
Connections:
- net +BATT: now also F2.1
- net GND: now also J5.1 (Pin_1)
- new net: F1.2, F2.2, J5.2 (Pin_2)
- new net +V_PWR: F1.1
Changed lines of the file:
@@
 	8100 3850 9100 3850
 $Sheet
-S 3450 5100 1300 1450
+S 3600 5200 1300 1450
 U 5EF5B1D1
 F0 "Power" 50
 F1 "power.sch" 50
-F2 "EN_12V" I L 3450 6100 50
-F3 "EN_3V3" I L 3450 6350 50
-F4 "VIN" I L 3450 5300 50
-F5 "12V" O R 4750 5300 50
-F6 "3V3" O R 4750 5700 50
-F7 "12V_STBY" O R 4750 5450 50
-F8 "3V3_STBY" O R 4750 5850 50
-F9 "3V0" O R 4750 6100 50
-F10 "2V5_REF" O R 4750 6350 50
+F2 "EN_12V" I L 3600 6200 50
+F3 "EN_3V3" I L 3600 6450 50
+F4 "VIN" I L 3600 5400 50
+F5 "12V" O R 4900 5400 50
+F6 "3V3" O R 4900 5800 50
+F7 "12V_STBY" O R 4900 5550 50
+F8 "3V3_STBY" O R 4900 5950 50
+F9 "3V0" O R 4900 6200 50
+F10 "2V5_REF" O R 4900 6450 50
 $EndSheet
 $Comp
 L power:+12V #PWR02
 U 1 1 5EF9721E
-P 4900 5300
-F 0 "#PWR02" H 4900 5150 50  0001 C CNN
-F 1 "+12V" H 4915 5473 50  0000 C CNN
-F 2 "" H 4900 5300 50  0001 C CNN
-F 3 "" H 4900 5300 50  0001 C CNN
-	1    4900 5300
-	1    0    0    -1
-$EndComp
-Wire Wire Line
-	4750 5300 4900 5300
-Text GLabel 4900 6350 2    50   Output ~ 0
+P 5050 5400
+F 0 "#PWR02" H 5050 5250 50  0001 C CNN
+F 1 "+12V" H 5065 5573 50  0000 C CNN
+F 2 "" H 5050 5400 50  0001 C CNN
+F 3 "" H 5050 5400 50  0001 C CNN
+	1    5050 5400
+	1    0    0    -1
+$EndComp
+Wire Wire Line
+	4900 5400 5050 5400
+Text GLabel 5050 6450 2    50   Output ~ 0
 VREF
 Wire Wire Line
-	4750 6350 4900 6350
+	4900 6450 5050 6450
 $Comp
 L power:+BATT #PWR01
 U 1 1 5EF9882C
-P 3250 5300
-F 0 "#PWR01" H 3250 5150 50  0001 C CNN
-F 1 "+BATT" H 3265 5473 50  0000 C CNN
-F 2 "" H 3250 5300 50  0001 C CNN
-F 3 "" H 3250 5300 50  0001 C CNN
-	1    3250 5300
-	1    0    0    -1
-$EndComp
-Wire Wire Line
-	3250 5300 3450 5300
-Wire Wire Line
-	4750 6100 4900 6100
+P 3400 5400
+F 0 "#PWR01" H 3400 5250 50  0001 C CNN
+F 1 "+BATT" H 3415 5573 50  0000 C CNN
+F 2 "" H 3400 5400 50  0001 C CNN
+F 3 "" H 3400 5400 50  0001 C CNN
+	1    3400 5400
+	1    0    0    -1
+$EndComp
+Wire Wire Line
+	3400 5400 3600 5400
+Wire Wire Line
+	4900 6200 5050 6200
 $Comp
 L power:+3V0 #PWR04
 U 1 1 5EF97D51
-P 4900 6100
-F 0 "#PWR04" H 4900 5950 50  0001 C CNN
-F 1 "+3V0" H 4915 6273 50  0000 C CNN
-F 2 "" H 4900 6100 50  0001 C CNN
-F 3 "" H 4900 6100 50  0001 C CNN
-	1    4900 6100
-	1    0    0    -1
-$EndComp
-Wire Wire Line
-	4750 5700 4900 5700
+P 5050 6200
+F 0 "#PWR04" H 5050 6050 50  0001 C CNN
+F 1 "+3V0" H 5065 6373 50  0000 C CNN
+F 2 "" H 5050 6200 50  0001 C CNN
+F 3 "" H 5050 6200 50  0001 C CNN
+	1    5050 6200
+	1    0    0    -1
+$EndComp
+Wire Wire Line
+	4900 5800 5050 5800
 $Comp
 L power:+3V3 #PWR03
 U 1 1 5EF979A2
-P 4900 5700
-F 0 "#PWR03" H 4900 5550 50  0001 C CNN
-F 1 "+3V3" H 4915 5873 50  0000 C CNN
-F 2 "" H 4900 5700 50  0001 C CNN
-F 3 "" H 4900 5700 50  0001 C CNN
-	1    4900 5700
-	1    0    0    -1
-$EndComp
-Wire Wire Line
-	5350 5450 5350 5300
-Wire Wire Line
-	4750 5450 5350 5450
-NoConn ~ 5350 5300
-Wire Wire Line
-	4750 5850 5350 5850
-Wire Wire Line
-	5350 5850 5350 5700
+P 5050 5800
+F 0 "#PWR03" H 5050 5650 50  0001 C CNN
+F 1 "+3V3" H 5065 5973 50  0000 C CNN
+F 2 "" H 5050 5800 50  0001 C CNN
+F 3 "" H 5050 5800 50  0001 C CNN
+	1    5050 5800
+	1    0    0    -1
+$EndComp
+Wire Wire Line
+	5500 5550 5500 5400
+Wire Wire Line
+	4900 5550 5500 5550
+NoConn ~ 5500 5400
+Wire Wire Line
+	4900 5950 5500 5950
+Wire Wire Line
+	5500 5950 5500 5800
 $Sheet
 S 3350 2050 1550 2200
@@
 F18 "CHB_TEMP" I R 4900 3900 50
 F19 "BAT_VOL" I L 3350 2200 50
+F20 "EN_12V" O L 3350 4100 50
+F21 "EN_3V3" O L 3350 4000 50
 $EndSheet
 $Comp
@@
 L Station:+3V3_STBY #PWR037
 U 1 1 5F0886C8
-P 5350 5700
-F 0 "#PWR037" H 5350 5550 50  0001 C CNN
-F 1 "+3V3_STBY" H 5365 5873 50  0000 C CNN
-F 2 "" H 5350 5700 50  0001 C CNN
-F 3 "" H 5350 5700 50  0001 C CNN
-	1    5350 5700
+P 5500 5800
+F 0 "#PWR037" H 5500 5650 50  0001 C CNN
+F 1 "+3V3_STBY" H 5515 5973 50  0000 C CNN
+F 2 "" H 5500 5800 50  0001 C CNN
+F 3 "" H 5500 5800 50  0001 C CNN
+	1    5500 5800
 	1    0    0    -1
 $EndComp
@@
 Wire Wire Line
 	2850 2200 2850 2250
+$Comp
+L Connector:Screw_Terminal_01x02 J5
+U 1 1 606EE99B
+P 1750 6100
+F 0 "J5" H 1668 6225 50  0000 C CNN
+F 1 "Screw_Terminal_01x02" H 1668 6226 50  0001 C CNN
+F 2 "TerminalBlock:TerminalBlock_bornier-2_P5.08mm" H 1750 6100 50  0001 C CNN
+F 3 "~" H 1750 6100 50  0001 C CNN
+	1    1750 6100
+	-1   0    0    1
+$EndComp
+$Comp
+L Station:+V_PWR #PWR029
+U 1 1 606F016B
+P 2150 5600
+F 0 "#PWR029" H 2150 5450 50  0001 C CNN
+F 1 "+V_PWR" H 2165 5773 50  0000 C CNN
+F 2 "" H 2150 5600 50  0001 C CNN
+F 3 "" H 2150 5600 50  0001 C CNN
+	1    2150 5600
+	1    0    0    -1
+$EndComp
+$Comp
+L power:+BATT #PWR049
+U 1 1 606F0A8F
+P 2500 5600
+F 0 "#PWR049" H 2500 5450 50  0001 C CNN
+F 1 "+BATT" H 2515 5773 50  0000 C CNN
+F 2 "" H 2500 5600 50  0001 C CNN
+F 3 "" H 2500 5600 50  0001 C CNN
+	1    2500 5600
+	1    0    0    -1
+$EndComp
+$Comp
+L power:GND #PWR013
+U 1 1 606F1060
+P 2050 6200
+F 0 "#PWR013" H 2050 5950 50  0001 C CNN
+F 1 "GND" H 2055 6027 50  0000 C CNN
+F 2 "" H 2050 6200 50  0001 C CNN
+F 3 "" H 2050 6200 50  0001 C CNN
+	1    2050 6200
+	1    0    0    -1
+$EndComp
+Wire Wire Line
+	1950 6100 2050 6100
+Wire Wire Line
+	2050 6100 2050 6200
+$Comp
+L Device:Fuse F1
+U 1 1 606F9313
+P 2150 5800
+F 0 "F1" H 2210 5800 50  0000 L CNN
+F 1 "Fuse" H 2210 5755 50  0001 L CNN
+F 2 "station:Fuse_2410" V 2080 5800 50  0001 C CNN
+F 3 "~" H 2150 5800 50  0001 C CNN
+	1    2150 5800
+	1    0    0    -1
+$EndComp
+$Comp
+L Device:Fuse F2
+U 1 1 606F9860
+P 2500 5800
+F 0 "F2" H 2560 5800 50  0000 L CNN
+F 1 "Fuse" H 2560 5755 50  0001 L CNN
+F 2 "Fuse:Fuse_1206_3216Metric" V 2430 5800 50  0001 C CNN
+F 3 "~" H 2500 5800 50  0001 C CNN
+	1    2500 5800
+	1    0    0    -1
+$EndComp
+Wire Wire Line
+	1950 6000 2150 6000
+Wire Wire Line
+	2150 6000 2150 5950
+Wire Wire Line
+	2150 6000 2500 6000
+Wire Wire Line
+	2500 6000 2500 5950
+Connection ~ 2150 6000
+Wire Wire Line
+	2500 5600 2500 5650
+Wire Wire Line
+	2150 5600 2150 5650
+Wire Wire Line
+	3350 4100 3150 4100
+Wire Wire Line
+	3150 4100 3150 6200
+Wire Wire Line
+	3150 6200 3600 6200
+Wire Wire Line
+	3350 4000 3050 4000
+Wire Wire Line
+	3050 4000 3050 6450
+Wire Wire Line
+	3050 6450 3600 6450
 $EndSCHEMATC

Commit message: Update BOM * Datasheets * Manufacturers * Part numbers
Parts:
- F1: Manufacturer (none) -> Eaton; Part Number (none) -> CB61F15A-TR2
- F2: Manufacturer (none) -> Bel Fuse Inc; Part Number (none) -> C1F 375
- J1, J2: Manufacturer (none) -> Adam Tech; Part Number (none) -> ASJ-125-3
- J3: Manufacturer (none) -> Amphenol; Part Number (none) -> 10129382-910002BLF
- J5: Manufacturer (none) -> CUI Devices; Part Number (none) -> TB004-508-02BE
- R61: Manufacturer (none) -> Panasonic; Part Number (none) -> ERJ-3EKF2004V; Tolerance (none) -> 1%
- R62: Manufacturer (none) -> Stackpole Electronics Inc; Part Number (none) -> RMCF0603FT120K; Tolerance (none) -> 1%
Changed lines of the file:
@@
 F 1 "AudioJack3" H 9020 2574 50  0000 R CNN
 F 2 "station:Jack_3.5mm_Adam_Tech_ASJ-125-3" H 9300 2550 50  0001 C CNN
-F 3 "~" H 9300 2550 50  0001 C CNN
+F 3 "https://app.adam-tech.com/products/download/data_sheet/203685/asj-125-3-data-sheet.pdf" H 9300 2550 50  0001 C CNN
+F 4 "Adam Tech" H 9300 2550 50  0001 C CNN "Manufacturer"
+F 5 "ASJ-125-3" H 9300 2550 50  0001 C CNN "Part Number"
 	1    9300 2550
 	-1   0    0    1
@@
 F 1 "AudioJack3" H 9020 3874 50  0000 R CNN
 F 2 "station:Jack_3.5mm_Adam_Tech_ASJ-125-3" H 9300 3850 50  0001 C CNN
-F 3 "~" H 9300 3850 50  0001 C CNN
+F 3 "https://app.adam-tech.com/products/download/data_sheet/203685/asj-125-3-data-sheet.pdf" H 9300 3850 50  0001 C CNN
+F 4 "Adam Tech" H 9300 3850 50  0001 C CNN "Manufacturer"
+F 5 "ASJ-125-3" H 9300 3850 50  0001 C CNN "Part Number"
 	1    9300 3850
 	-1   0    0    1
@@
 F 1 "Conn_02x05_Odd_Even" H 5650 2926 50  0001 C CNN
 F 2 "station:PinHeader_2x05_P2.54mm_BoardEdge" H 5600 2600 50  0001 C CNN
-F 3 "~" H 5600 2600 50  0001 C CNN
+F 3 "https://cdn.amphenol-icc.com/media/wysiwyg/files/drawing/10129382.pdf" H 5600 2600 50  0001 C CNN
+F 4 "Amphenol" H 5600 2600 50  0001 C CNN "Manufacturer"
+F 5 "10129382-910002BLF" H 5600 2600 50  0001 C CNN "Part Number"
 	1    5600 2600
 	1    0    0    -1
@@
 F 1 "2M" H 2920 1955 50  0000 L CNN
 F 2 "Resistor_SMD:R_0603_1608Metric" V 2780 2000 50  0001 C CNN
-F 3 "~" H 2850 2000 50  0001 C CNN
+F 3 "https://industrial.panasonic.com/cdbs/www-data/pdf/RDA0000/AOA0000C304.pdf" H 2850 2000 50  0001 C CNN
+F 4 "Panasonic" H 2850 2000 50  0001 C CNN "Manufacturer"
+F 5 "ERJ-3EKF2004V" H 2850 2000 50  0001 C CNN "Part Number"
+F 6 "1%" H 2850 2000 50  0001 C CNN "Tolerance"
 	1    2850 2000
 	1    0    0    -1
@@
 F 1 "120k" H 2920 2355 50  0000 L CNN
 F 2 "Resistor_SMD:R_0603_1608Metric" V 2780 2400 50  0001 C CNN
-F 3 "~" H 2850 2400 50  0001 C CNN
+F 3 "https://www.seielect.com/catalog/sei-packaging.pdf" H 2850 2400 50  0001 C CNN
+F 4 "Stackpole Electronics Inc" H 2850 2400 50  0001 C CNN "Manufacturer"
+F 5 "RMCF0603FT120K" H 2850 2400 50  0001 C CNN "Part Number"
+F 6 "1%" H 2850 2400 50  0001 C CNN "Tolerance"
 	1    2850 2400
 	1    0    0    -1
@@
 F 1 "Screw_Terminal_01x02" H 1668 6226 50  0001 C CNN
 F 2 "TerminalBlock:TerminalBlock_bornier-2_P5.08mm" H 1750 6100 50  0001 C CNN
-F 3 "~" H 1750 6100 50  0001 C CNN
+F 3 "https://www.cuidevices.com/product/resource/digikeypdf/tb004-508.pdf" H 1750 6100 50  0001 C CNN
+F 4 "CUI Devices" H 1750 6100 50  0001 C CNN "Manufacturer"
+F 5 "TB004-508-02BE" H 1750 6100 50  0001 C CNN "Part Number"
 	1    1750 6100
 	-1   0    0    1
@@
 F 1 "Fuse" H 2210 5755 50  0001 L CNN
 F 2 "station:Fuse_2410" V 2080 5800 50  0001 C CNN
-F 3 "~" H 2150 5800 50  0001 C CNN
+F 3 "https://www.eaton.com/content/dam/eaton/products/electronic-components/resources/data-sheet/eaton-cb61f-surface-mount-brick-fuses-data-sheet.pdf" H 2150 5800 50  0001 C CNN
+F 4 "Eaton" H 2150 5800 50  0001 C CNN "Manufacturer"
+F 5 "CB61F15A-TR2" H 2150 5800 50  0001 C CNN "Part Number"
 	1    2150 5800
 	1    0    0    -1
@@
 F 1 "Fuse" H 2560 5755 50  0001 L CNN
 F 2 "Fuse:Fuse_1206_3216Metric" V 2430 5800 50  0001 C CNN
-F 3 "~" H 2500 5800 50  0001 C CNN
+F 3 "https://belfuse.com/resources/datasheets/circuitprotection/ds-cp-c1f-series.pdf" H 2500 5800 50  0001 C CNN
+F 4 "Bel Fuse Inc" H 2500 5800 50  0001 C CNN "Manufacturer"
+F 5 "C1F 375" H 2500 5800 50  0001 C CNN "Part Number"
 	1    2500 5800
 	1    0    0    -1
